File: soroka-pcb/soroka.kicad_pcb (KiCad board)
At the start: 2 copper layers, 303.2 x 76.2 mm, 109 parts, among them SW1 MX150, SW10 MX100, SW11 MX100, SW12 MX100, SW13 MX100, SW14 MX100, SW15 Stepped, SW16 MX100, SW17 MX100, SW18 MX100, SW19 MX100, SW2 MX100, SW20 MX100, SW21 MX100, SW22 MX100, SW23 MX100, SW24 MX100, SW25 MX100, SW26 MX100, SW27 MX175, SW28 MX225R, SW29 MX100, SW3 MX100, SW30 MX100, SW31 MX100, SW32 MX100, SW33 MX100, SW34 MX100, SW35 MX100, SW36 MX100, SW37 MX100, SW38 MX100, SW39 1.25u, SW4 MX100, SW40 2.25u, SW41 1u, SW42 MX125, SW43 MX125, SW44 MX125, SW45 MX100, SW46 3u, SW47 2.25u, SW48 7u/1u, SW49 3u, SW5 MX100, SW50 MX100, SW51 MX125, SW52 MX125, SW53 MX125, SW54 2.75u, SW55 1.75u, SW55 RotaryEncoder_Switch, SW6 MX100, SW7 MX100, SW8 MX100, SW9 MX100, U1 RP2040-Zero

Commit message: fixed typo and created new production files
Other:
- board text added: "MCU on this side!"
- board text removed: "MSU on this side!"
Changed lines of the file:
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@@
     )
   )
-  (gr_text "MSU on this side!" (at 376.36875 65.42125 90) (layer "B.SilkS")
+  (gr_text "MCU on this side!" (at 376.36875 65.42125 90) (layer "B.SilkS")
     (effects (font (size 1 1) (thickness 0.15) italic) (justify left bottom mirror))
   )
@@
       2b125c96-5938-42af-b563-25285dc0173c
       7822fc7b-0ddd-4789-913a-2ae969f25fa8
-      f09475d9-3ac7-4f5a-a34c-41e4d01c9abd
     )
   )
