File: v2/soroka-v2-pcb-HS/soroka.kicad_pcb (KiCad board)
At the start: 2 copper layers, 305.2 x 76.2 mm, 108 parts, among them SW1 MX150H, SW10 MXSwitch, SW11 MXSwitch, SW12 MXSwitch, SW13 MXSwitch, SW14 MXSwitch, SW15 Normal, SW16 MXSwitch, SW17 MXSwitch, SW18 MXSwitch, SW19 MXSwitch, SW2 MXSwitch, SW20 MXSwitch, SW21 MXSwitch, SW22 MXSwitch, SW23 MXSwitch, SW24 MXSwitch, SW25 MXSwitch, SW26 MXSwitch, SW27 MX175H, SW28 MX225R, SW29 MXSwitch, SW3 MXSwitch, SW30 MXSwitch, SW31 MXSwitch, SW32 MXSwitch, SW33 MXSwitch, SW34 MXSwitch, SW35 MXSwitch, SW36 MXSwitch, SW37 MXSwitch, SW38 MXSwitch, SW39 1.25u, SW4 MXSwitch, SW41 1u, SW42 MXH125, SW43 MXH125, SW44 MXH125, SW45 MXSwitch, SW46 Stepped, SW47 2.25u, SW48 7u, SW5 MXSwitch, SW50 MXSwitch, SW51 MXH125, SW52 MXH125, SW53 MXH125, SW54 2.75u, SW55 RotaryEncoder_Switch, SW56 RotaryEncoder_Switch, SW6 MXSwitch, SW7 MXSwitch, SW8 MXSwitch, SW9 MXSwitch

Commit message: added untested hotswap PCB
Parts:
- removed H1, H10, H11, H12, H2, H3, H4, H5, H6, H7, H8, H9: MountingHole, kapee-keeb-parts:MountingHole_2.2mm_M2_DIN965_Pad
- ? (x12), MP: footprint kapee-keeb-parts: -> Library:
- D1, D10, D11, D12, D13, D14, D15, D16, D17, D18, D19, D2, D20, D21, D22, D23, D24, D25, D26, D27, D3, D4, D5, D6, D7, D8, D9: footprint Package_TO_SOT_SMD:SOT-23 -> Library:SOT-23
- G***: footprint LOGO -> Library:LOGO
- RZ1: footprint kapee-keeb-parts:MCU_rp2040-zero-tht -> Library:MCU_rp2040-zero-tht
- SW55: footprint kapee-keeb-parts:RotaryEncoder_Alps_EC11E-Switch_Vertical_H20mm -> Library:RotaryEncoder_Alps_EC11E-Switch_Vertical_H20mm
- SW56: footprint kapee-keeb-parts:EVQWGD001 -> Library:EVQWGD001
- moved D24 7.40 mm to (353.6, 116.8)
Routing:
- net COL0: track 103.8 -> 366.2 mm, vias 4 -> 5
- net COL1: track 86.8 -> 329.9 mm, vias 4 -> 5
- net COL2: track 78.7 -> 300.4 mm, vias 4 -> 5
- net COL3: track 78.0 -> 283.3 mm, vias 4 -> 5
- net COL4: track 74.8 -> 269.3 mm, vias 4 -> 5
- net COL5: track 53.0 -> 230.7 mm, vias 3 -> 4
- net COL6: track 78.0 -> 239.2 mm, vias 4 -> 5
- net COL7: track 53.0 -> 197.7 mm, vias 3 -> 4
- net COL12: track 25.0 -> 152.5 mm, vias 2 -> 4
- net COL8: track 96.1 -> 223.4 mm, vias 4 -> 5
- net COL9: track 78.0 -> 189.0 mm, vias 4 -> 5
- net COL10: track 76.8 -> 172.8 mm, vias 4 -> 5
- net ROW2: track 229.3 -> 314.2 mm
- net ENC_CCW: track 0.00 -> 81.3 mm
- net COL11: track 77.0 -> 157.2 mm, vias 4 -> 5
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Other:
- board text added: "7"
- board text added: "Regular"
- board text added: "Stepped"
- board text added: "soroka | 2025"
- board text removed: "3V"
- board text removed: "kapee!"
